File: ethernet.kicad_sch (KiCad schematic)
At the start: 25 parts, among them J12 RJ45_Hanrun_HR911105A_Horizon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, U7 LAN8742A, Y3 25Mhz

Commit message: style: 修改图框
Other:
- title: (none) -> 以太网组件
Changed lines of the file:
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@@
 	(paper "A5")
 	(title_block
-		(date "2026-06-08")
+		(title "以太网组件")
+		(date "2026-06-10")
+		(rev "V0.0.1")
 		(company "重庆创迪科技发展有限公司")
 	)

Commit message: feat: 添加了安装孔
Parts:
- renumbered J12 to J11
Changed lines of the file:
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@@
 		(in_pos_files yes)
 		(dnp no)
-		(property "Reference" "#PWR058"
+		(property "Reference" "#PWR057"
 			(at 190.5 71.12 0)
 			(hide yes)
@@
 			(project "通用型控制卡"
 				(path "/663e394a-ab41-456f-8927-f2089badb93c"
-					(reference "#PWR058")
+					(reference "#PWR057")
 					(unit 1)
 				)
@@
 		(in_pos_files yes)
 		(dnp no)
-		(property "Reference" "#PWR057"
+		(property "Reference" "#PWR056"
 			(at 38.1 40.64 0)
 			(hide yes)
@@
 			(project "通用型控制卡"
 				(path "/663e394a-ab41-456f-8927-f2089badb93c"
-					(reference "#PWR057")
+					(reference "#PWR056")
 					(unit 1)
 				)
@@
 		(in_pos_files yes)
 		(dnp no)
-		(property "Reference" "#PWR060"
+		(property "Reference" "#PWR059"
 			(at 113.03 83.82 0)
 			(hide yes)
@@
 			(project "通用型控制卡"
 				(path "/663e394a-ab41-456f-8927-f2089badb93c"
-					(reference "#PWR060")
+					(reference "#PWR059")
 					(unit 1)
 				)
@@
 		(in_pos_files yes)
 		(dnp no)
-		(property "Reference" "#PWR061"
+		(property "Reference" "#PWR060"
 			(at 19.05 100.33 0)
 			(hide yes)
@@
 			(project "通用型控制卡"
 				(path "/663e394a-ab41-456f-8927-f2089badb93c"
-					(reference "#PWR061")
+					(reference "#PWR060")
 					(unit 1)
 				)
@@
 		(in_pos_files yes)
 		(dnp no)
-		(property "Reference" "#PWR059"
+		(property "Reference" "#PWR058"
 			(at 163.83 82.55 0)
 			(hide yes)
@@
 			(project "通用型控制卡"
 				(path "/663e394a-ab41-456f-8927-f2089badb93c"
-					(reference "#PWR059")
+					(reference "#PWR058")
 					(unit 1)
 				)
@@
 		(in_pos_files yes)
 		(dnp no)
-		(property "Reference" "#PWR065"
+		(property "Reference" "#PWR064"
 			(at 31.75 132.08 0)
 			(hide yes)
@@
 			(project "通用型控制卡"
 				(path "/663e394a-ab41-456f-8927-f2089badb93c"
-					(reference "#PWR065")
+					(reference "#PWR064")
 					(unit 1)
 				)
@@
 		(in_pos_files yes)
 		(dnp no)
-		(property "Reference" "#PWR055"
+		(property "Reference" "#PWR054"
 			(at 57.15 31.75 0)
 			(hide yes)
@@
 			(project "通用型控制卡"
 				(path "/663e394a-ab41-456f-8927-f2089badb93c"
-					(reference "#PWR055")
+					(reference "#PWR054")
 					(unit 1)
 				)
@@
 		(in_pos_files yes)
 		(dnp no)
-		(property "Reference" "#PWR063"
+		(property "Reference" "#PWR062"
 			(at 31.75 107.95 0)
 			(hide yes)
@@
 			(project "通用型控制卡"
 				(path "/663e394a-ab41-456f-8927-f2089badb93c"
-					(reference "#PWR063")
+					(reference "#PWR062")
 					(unit 1)
 				)
@@
 		(dnp no)
 		(fields_autoplaced yes)
-		(property "Reference" "J12"
+		(property "Reference" "J11"
 			(at 154.94 44.45 0)
 			(show_name no)
@@
 			(project "通用型控制卡"
 				(path "/663e394a-ab41-456f-8927-f2089badb93c"
-					(reference "J12")
+					(reference "J11")
 					(unit 1)
 				)
@@
 		(in_pos_files yes)
 		(dnp no)
-		(property "Reference" "#PWR054"
+		(property "Reference" "#PWR053"
 			(at 82.55 33.02 0)
 			(hide yes)
@@
 			(project "通用型控制卡"
 				(path "/663e394a-ab41-456f-8927-f2089badb93c"
-					(reference "#PWR054")
+					(reference "#PWR053")
 					(unit 1)
 				)
@@
 		(in_pos_files yes)
 		(dnp no)
-		(property "Reference" "#PWR062"
+		(property "Reference" "#PWR061"
 			(at 62.23 101.6 0)
 			(hide yes)
@@
 			(project "通用型控制卡"
 				(path "/663e394a-ab41-456f-8927-f2089badb93c"
-					(reference "#PWR062")
+					(reference "#PWR061")
 					(unit 1)
 				)
@@
 		(in_pos_files yes)
 		(dnp no)
-		(property "Reference" "#PWR064"
+		(property "Reference" "#PWR063"
 			(at 72.39 116.84 0)
 			(hide yes)
@@
 			(project "通用型控制卡"
 				(path "/663e394a-ab41-456f-8927-f2089badb93c"
-					(reference "#PWR064")
+					(reference "#PWR063")
 					(unit 1)
 				)
@@
 		(in_pos_files yes)
 		(dnp no)
-		(property "Reference" "#PWR056"
+		(property "Reference" "#PWR055"
 			(at 62.23 34.29 0)
 			(hide yes)
@@
 			(project "通用型控制卡"
 				(path "/663e394a-ab41-456f-8927-f2089badb93c"
-					(reference "#PWR056")
-					(unit 1)
-				)
+					(reference "#PWR055")
+					(unit 1)
+				)
