File: ethernet.kicad_sch (KiCad schematic)
At the start: 25 parts, among them J11 RJ45_Hanrun_HR911105A_Horizon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, U7 LAN8742A, Y3 25Mhz

Commit message: feat: 布局完成，正在布线
Parts:
- J11: footprint Connector_RJ:RJ45_Hanrun_HR911105A_Horizontal -> wyh:RJ45_Hanrun_HR911105A_Horizontal
- U7: footprint Package_DFN_QFN:VQFN-24-1EP_4x4mm_P0.5mm_EP2.5x2.5mm_ThermalVias -> wyh:VQFN-24-1EP_4x4mm_P0.5mm_EP2.5x2.5mm_ThermalVias
- Y3: footprint Crystal:Crystal_SMD_3225-4Pin_3.2x2.5mm_HandSoldering -> Crystal:Crystal_SMD_3225-4Pin_3.2x2.5mm
Connections:
- net RJ45_RX+: now also R20.2
- net RJ45_TX-: no longer R20.2
Other:
- note added: "Tips: 差分信号对内长度控制在5mil以内，对间长度控制在50mil以内，阻抗控制在100Ω"
