File: serial_port.kicad_sch (KiCad schematic)
At the start: 30 parts, among them J10 RS232_1, J11 RS232_2, J8 RS485_1, J9 RS485_2, U4 MAX13487EESA+T, U5 MAX13487EESA+T, U6 MAX3232

Commit message: style: 修改图框
Other:
- title: (none) -> 串口通讯组件
Changed lines of the file:
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@@
 	(paper "A4")
 	(title_block
-		(date "2026-06-08")
+		(title "串口通讯组件")
+		(date "2026-06-10")
+		(rev "V0.0.1")
 		(company "重庆创迪科技发展有限公司")
 	)

Commit message: feat: 添加了安装孔
Parts:
- renumbered J11 to J10, J8 to J7, J9 to J8, J10 to J9
Changed lines of the file:
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@@
 		(in_pos_files yes)
 		(dnp no)
-		(property "Reference" "#PWR047"
+		(property "Reference" "#PWR046"
 			(at 111.76 88.9 0)
 			(hide yes)
@@
 			(project "通用型控制卡"
 				(path "/3cb67af0-7388-47d7-b8d2-13d3ce4998ce"
-					(reference "#PWR047")
+					(reference "#PWR046")
 					(unit 1)
 				)
@@
 		(in_pos_files yes)
 		(dnp no)
-		(property "Reference" "#PWR046"
+		(property "Reference" "#PWR045"
 			(at 200.66 87.63 0)
 			(hide yes)
@@
 			(project "通用型控制卡"
 				(path "/3cb67af0-7388-47d7-b8d2-13d3ce4998ce"
-					(reference "#PWR046")
+					(reference "#PWR045")
 					(unit 1)
 				)
@@
 		(in_pos_files yes)
 		(dnp no)
-		(property "Reference" "J11"
+		(property "Reference" "J10"
 			(at 147.574 163.576 0)
 			(show_name no)
@@
 			(project "通用型控制卡"
 				(path "/3cb67af0-7388-47d7-b8d2-13d3ce4998ce"
-					(reference "J11")
+					(reference "J10")
 					(unit 1)
 				)
@@
 		(in_pos_files yes)
 		(dnp no)
-		(property "Reference" "#PWR051"
+		(property "Reference" "#PWR050"
 			(at 100.33 156.21 0)
 			(hide yes)
@@
 			(project "通用型控制卡"
 				(path "/3cb67af0-7388-47d7-b8d2-13d3ce4998ce"
-					(reference "#PWR051")
+					(reference "#PWR050")
 					(unit 1)
 				)
@@
 		(in_pos_files yes)
 		(dnp no)
-		(property "Reference" "#PWR044"
+		(property "Reference" "#PWR043"
 			(at 251.46 73.66 0)
 			(hide yes)
@@
 			(project "通用型控制卡"
 				(path "/3cb67af0-7388-47d7-b8d2-13d3ce4998ce"
-					(reference "#PWR044")
+					(reference "#PWR043")
 					(unit 1)
 				)
@@
 		(in_pos_files yes)
 		(dnp no)
-		(property "Reference" "#PWR053"
+		(property "Reference" "#PWR052"
 			(at 69.85 189.23 0)
 			(hide yes)
@@
 			(project "通用型控制卡"
 				(path "/3cb67af0-7388-47d7-b8d2-13d3ce4998ce"
-					(reference "#PWR053")
+					(reference "#PWR052")
 					(unit 1)
 				)
@@
 		(in_pos_files yes)
 		(dnp no)
-		(property "Reference" "#PWR052"
+		(property "Reference" "#PWR051"
 			(at 99.06 185.42 0)
 			(hide yes)
@@
 			(project "通用型控制卡"
 				(path "/3cb67af0-7388-47d7-b8d2-13d3ce4998ce"
-					(reference "#PWR052")
+					(reference "#PWR051")
 					(unit 1)
 				)
@@
 		(in_pos_files yes)
 		(dnp no)
-		(property "Reference" "#PWR041"
+		(property "Reference" "#PWR040"
 			(at 62.23 40.64 0)
 			(hide yes)
@@
 			(project "通用型控制卡"
 				(path "/3cb67af0-7388-47d7-b8d2-13d3ce4998ce"
-					(reference "#PWR041")
+					(reference "#PWR040")
 					(unit 1)
 				)
@@
 		(in_pos_files yes)
 		(dnp no)
-		(property "Reference" "#PWR042"
+		(property "Reference" "#PWR041"
 			(at 200.66 40.64 0)
 			(hide yes)
@@
 			(project "通用型控制卡"
 				(path "/3cb67af0-7388-47d7-b8d2-13d3ce4998ce"
-					(reference "#PWR042")
+					(reference "#PWR041")
 					(unit 1)
 				)
@@
 		(in_pos_files yes)
 		(dnp no)
-		(property "Reference" "#PWR049"
+		(property "Reference" "#PWR048"
 			(at 69.85 121.92 0)
 			(hide yes)
@@
 			(project "通用型控制卡"
 				(path "/3cb67af0-7388-47d7-b8d2-13d3ce4998ce"
-					(reference "#PWR049")
+					(reference "#PWR048")
 					(unit 1)
 				)
@@
 		(in_pos_files yes)
 		(dnp no)
-		(property "Reference" "#PWR043"
+		(property "Reference" "#PWR042"
 			(at 111.76 73.66 0)
 			(hide yes)
@@
 			(project "通用型控制卡"
 				(path "/3cb67af0-7388-47d7-b8d2-13d3ce4998ce"
-					(reference "#PWR043")
+					(reference "#PWR042")
 					(unit 1)
 				)
@@
 		(in_pos_files yes)
 		(dnp no)
-		(property "Reference" "#PWR045"
+		(property "Reference" "#PWR044"
 			(at 62.23 87.63 0)
 			(hide yes)
@@
 			(project "通用型控制卡"
 				(path "/3cb67af0-7388-47d7-b8d2-13d3ce4998ce"
-					(reference "#PWR045")
+					(reference "#PWR044")
 					(unit 1)
 				)
@@
 		(in_pos_files yes)
 		(dnp no)
-		(property "Reference" "J8"
+		(property "Reference" "J7"
 			(at 106.68 49.53 0)
 			(show_name no)
@@
 			(project "通用型控制卡"
 				(path "/3cb67af0-7388-47d7-b8d2-13d3ce4998ce"
-					(reference "J8")
+					(reference "J7")
 					(unit 1)
 				)
@@
 		(in_pos_files yes)
 		(dnp no)
-		(property "Reference" "#PWR048"
+		(property "Reference" "#PWR047"
 			(at 251.46 88.9 0)
 			(hide yes)
@@
 			(project "通用型控制卡"
 				(path "/3cb67af0-7388-47d7-b8d2-13d3ce4998ce"
-					(reference "#PWR048")
+					(reference "#PWR047")
 					(unit 1)
 				)
@@
 		(in_pos_files yes)
 		(dnp no)
-		(property "Reference" "#PWR050"
+		(property "Reference" "#PWR049"
 			(at 60.96 125.73 0)
 			(hide yes)
@@
 			(project "通用型控制卡"
 				(path "/3cb67af0-7388-47d7-b8d2-13d3ce4998ce"
-					(reference "#PWR050")
+					(reference "#PWR049")
 					(unit 1)
 				)
@@
 		(in_pos_files yes)
 		(dnp no)
-		(property "Reference" "J9"
+		(property "Reference" "J8"
 			(at 242.824 49.276 0)
 			(show_name no)
@@
 			(project "通用型控制卡"
 				(path "/3cb67af0-7388-47d7-b8d2-13d3ce4998ce"
-					(reference "J9")
+					(reference "J8")
 					(unit 1)
 				)
@@
 		(in_pos_files yes)
 		(dnp no)
-		(property "Reference" "J10"
+		(property "Reference" "J9"
 			(at 147.32 156.21 0)
 			(show_name no)
@@
 			(project "通用型控制卡"
 				(path "/3cb67af0-7388-47d7-b8d2-13d3ce4998ce"
-					(reference "J10")
+					(reference "J9")
 					(unit 1)
 				)
