File: serial_port.kicad_sch (KiCad schematic)
At the start: 30 parts, among them J10 RS232_2, J7 RS485_1, J8 RS485_2, J9 RS232_1, U4 MAX13487EESA+T, U5 MAX13487EESA+T, U6 MAX3232

Commit message: 根据BOM表调整部分元件封装
Parts:
- C36, C37, C38, C39: footprint Capacitor_SMD:C_0402_1005Metric_Pad0.74x0.62mm_HandSolder -> Capacitor_SMD:C_0603_1608Metric_Pad1.08x0.95mm_HandSolder
- J10: value RS232_2 -> Sockets; 定义 (none) -> RS232_2
- J7: value RS485_1 -> Sockets; 定义 (none) -> RS485_1
- J8: value RS485_2 -> Sockets; 定义 (none) -> RS485_2
- J9: value RS232_1 -> Sockets; 定义 (none) -> RS232_1
Changed lines of the file:
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@@
 			)
 		)
-		(property "Footprint" "Capacitor_SMD:C_0402_1005Metric_Pad0.74x0.62mm_HandSolder"
+		(property "Footprint" "Capacitor_SMD:C_0603_1608Metric_Pad1.08x0.95mm_HandSolder"
 			(at 105.1052 80.01 0)
 			(hide yes)
@@
 			)
 		)
-		(property "Footprint" "Capacitor_SMD:C_0402_1005Metric_Pad0.74x0.62mm_HandSolder"
+		(property "Footprint" "Capacitor_SMD:C_0603_1608Metric_Pad1.08x0.95mm_HandSolder"
 			(at 112.7252 80.01 0)
 			(hide yes)
@@
 			)
 		)
-		(property "Footprint" "Capacitor_SMD:C_0402_1005Metric_Pad0.74x0.62mm_HandSolder"
+		(property "Footprint" "Capacitor_SMD:C_0603_1608Metric_Pad1.08x0.95mm_HandSolder"
 			(at 252.4252 80.01 0)
 			(hide yes)
@@
 		(dnp no)
 		(property "Reference" "J10"
-			(at 147.574 163.576 0)
+			(at 147.066 163.83 0)
 			(show_name no)
 			(do_not_autoplace no)
@@
 			)
 		)
-		(property "Value" "RS232_2"
-			(at 147.574 166.116 0)
+		(property "Value" "Sockets"
+			(at 147.066 166.116 0)
+			(hide yes)
 			(show_name no)
 			(do_not_autoplace no)
@@
 			)
 		)
+		(property "定义" "RS232_2"
+			(at 151.13 166.37 0)
+			(show_name no)
+			(do_not_autoplace no)
+			(effects
+				(font
+					(size 1.27 1.27)
+				)
+			)
+		)
 		(pin "1"
 		)
@@
 			)
 		)
-		(property "Footprint" "Capacitor_SMD:C_0402_1005Metric_Pad0.74x0.62mm_HandSolder"
+		(property "Footprint" "Capacitor_SMD:C_0603_1608Metric_Pad1.08x0.95mm_HandSolder"
 			(at 244.8052 80.01 0)
 			(hide yes)
@@
 		(dnp no)
 		(property "Reference" "J7"
-			(at 106.68 49.53 0)
+			(at 106.426 49.53 0)
 			(show_name no)
 			(do_not_autoplace no)
@@
 			)
 		)
-		(property "Value" "RS485_1"
+		(property "Value" "Sockets"
 			(at 106.68 52.07 0)
+			(hide yes)
 			(show_name no)
 			(do_not_autoplace no)
@@
 			)
 		)
+		(property "定义" "RS485_1"
+			(at 110.49 52.07 0)
+			(show_name no)
+			(do_not_autoplace no)
+			(effects
+				(font
+					(size 1.27 1.27)
+				)
+			)
+		)
 		(pin "1"
 		)
@@
 		(dnp no)
 		(property "Reference" "J8"
-			(at 242.824 49.276 0)
+			(at 242.316 49.53 0)
 			(show_name no)
 			(do_not_autoplace no)
@@
 			)
 		)
-		(property "Value" "RS485_2"
+		(property "Value" "Sockets"
 			(at 242.824 51.816 0)
+			(hide yes)
 			(show_name no)
 			(do_not_autoplace no)
@@
 			)
 		)
+		(property "定义" "RS485_2"
+			(at 246.38 52.07 0)
+			(show_name no)
+			(do_not_autoplace no)
+			(effects
+				(font
+					(size 1.27 1.27)
+				)
+			)
+		)
 		(pin "1"
 		)
@@
 			)
 		)
-		(property "Value" "RS232_1"
+		(property "Value" "Sockets"
 			(at 147.32 158.75 0)
+			(hide yes)
 			(show_name no)
 			(do_not_autoplace no)
@@
 			(show_name no)
 			(do_not_autoplace no)
+			(effects
+				(font
+					(size 1.27 1.27)
+				)
+			)
+		)
+		(property "定义" "RS232_1"
+			(at 151.13 158.75 0)
+			(show_name no)
+			(do_not_autoplace no)

Commit message: fix: 修改了485芯片的封装，添加了保险丝的封装
Parts:
- U4, U5: footprint Package_SO:SOIC-8_5.3x5.3mm_P1.27mm -> Package_SO:SOIC-8_3.9x4.9mm_P1.27mm
Changed lines of the file:
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@@
 			)
 		)
-		(property "Footprint" "Package_SO:SOIC-8_5.3x5.3mm_P1.27mm"
+		(property "Footprint" "Package_SO:SOIC-8_3.9x4.9mm_P1.27mm"
 			(at 200.66 57.15 0)
 			(hide yes)
@@
 			)
 		)
-		(property "Footprint" "Package_SO:SOIC-8_5.3x5.3mm_P1.27mm"
+		(property "Footprint" "Package_SO:SOIC-8_3.9x4.9mm_P1.27mm"
 			(at 62.23 57.15 0)
 			(hide yes)
