File: 通用型控制卡.kicad_sch (KiCad schematic)
At the start: 68 parts, among them J1 EXT, J2 HUB75_A, J3 HUB75_B, J4 PWR, J5 SWD_TC2030, J6 SWD_IDC, J7 DBG_Serial, SW1 RESET, SW2 TST_KEY, U1 STM32H753IITx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

Commit message: style: 修改图框
Other:
- title: (none) -> MCU及连接器组件
Changed lines of the file:
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@@
 	(paper "A3")
 	(title_block
-		(date "2026-06-08")
+		(title "MCU及连接器组件")
+		(date "2026-06-10")
+		(rev "V0.0.1")
 		(company "重庆创迪科技发展有限公司")
 	)
@@
 	)
 	(embedded_fonts no)
+	(embedded_files
+		(file
+			(name "通用图框1.kicad_wks")
+			(type worksheet)
+			(data |KLUv/WD/B8USAPbbVyEQtRtqMSSdbV9NJOgutWcFuLtYyEKEJnfhgyYigNABwAFOAEgAUADf4dgs
+				Z1/Lydun/ca9Qp1Rduc1VuTXeoUaZ3vJhj/yJwAAAQEIeg9llJPSKKtxzQOpzvi37Nc5hcScs6KS
+				9sU2zB4iAAKC8CPSNFtnP4RVpS0raZS7a/s3B71l9ptx917LltSnwx7X7r399s635oJw3prqv/59
+				uKNNW3OdUimjNdtKWNGSsz9vH1JU+7fd7zx/+B9zIA7tsGJlJSKSrELBMBrjWmQO04BKaYiIrrHW
+				E2a5GBp2qVQy06AV/hsj50zK/te7Jm3shyBPpT0vEq0tOY6TsyIA/uLN7Eo7xCA1qf6RP/dVBgFB
+				odZq1pog3Q388KLGOTORawKRLKpJpawiAnJFsEfWsA1DjZTGw8QelszivbVYVv/2Zbzp7OA2oWCT
+				a+IlWzHEOduSM8NglJBTpKyxtpyTCmig0TyHIBoSEUmSJB1gRMQM1jYMIOfcsItWzD3szqgaUdxx
+				TgCQW4aJoZlYtE6g2ps1ozNiaWv22Ide/dY5FsqTIKSIC1ugFWQbzBGuo/D5YoXrzqo3b4IwiYN7
+				OLONr1nBoRNFbMuQcKm0N22S0SfWc0XdAj4DcEo6nz2qwzgdefJBv7I1DznaKLcRqLv01tYfGAS0
+				D1Pe6FD24hwH5J3TnaslBJLFLMa6M1/2BGprHZe2YeDyqCekB9pq0hViMAAn+rLCIUrMJoHOq88h
+				CmbvNEjubNFBQptT+a0IkPO+Y1ijQVNP3Jt1fSBYLmFjuevAHwNcBQ==|
+			)
+			(checksum "28357255A911CC7409421370E643CAAB")
+		)
+	)
 )

Commit message: feat: 添加了安装孔
Parts:
- removed J1: EXT, Connector_JST:JST_PUD_B32B-PUDSS_2x16_P2.00mm_Vertical, symbol Connector_Generic:Conn_02x16_Counter_Clockwise
- removed J6: SWD_IDC, Connector_IDC:IDC-Header_2x03_P2.54mm_Vertical, symbol Connector_Generic:Conn_02x03_Counter_Clockwise
- removed J7: DBG_Serial, Connector_JST:JST_XH_B4B-XH-A_1x04_P2.50mm_Vertical, symbol Connector:Conn_01x04_Pin
- added H1, H2, H3, H4: MountingHole_Pad, MountingHole:MountingHole_3.2mm_M3_Pad, symbol Mechanical:MountingHole_Pad
- added J13: EXT, Connector_IDC:IDC-Header_2x15_P2.54mm_Vertical, symbol Connector_Generic:Conn_02x15_Counter_Clockwise
- added J6: SWD_IDC, Connector_IDC:IDC-Header_2x04_P2.54mm_Vertical, symbol Connector_Generic:Conn_02x04_Counter_Clockwise
Connections:
- net +3V3: now also J13.30 (Pin_30), J6.8 (Pin_8)
- net +5V: now also J13.1 (Pin_1)
- net DBG_MCU_RX: now also J6.3 (Pin_3)
- net DBG_MCU_TX: now also J6.6 (Pin_6)
- net EX_FUN.IIC_SCL: now also J13.22 (Pin_22)
- net EX_FUN.IIC_SDA: now also J13.23 (Pin_23)
- net EX_FUN.SPI_MISO: now also J13.20 (Pin_20)
- net EX_FUN.SPI_MOSI: now also J13.21 (Pin_21)
- net EX_FUN.SPI_NSS: now also J13.18 (Pin_18)
- net EX_FUN.SPI_SCK: now also J13.19 (Pin_19)
- net EX_FUN.UART5_RX: now also J13.26 (Pin_26)
- net EX_FUN.UART5_TX: now also J13.27 (Pin_27)
- net EX_FUN.UART7_RX: now also J13.24 (Pin_24)
- net EX_FUN.UART7_TX: now also J13.25 (Pin_25)
- net EX_IO.ADC0: now also J13.12 (Pin_12)
- net EX_IO.ADC1: now also J13.13 (Pin_13)
- net EX_IO.ADC2: now also J13.14 (Pin_14)
- net EX_IO.ADC3: now also J13.17 (Pin_17)
- net EX_IO.IO0: now also J13.2 (Pin_2)
- net EX_IO.IO1: now also J13.3 (Pin_3)
- net EX_IO.IO2: now also J13.4 (Pin_4)
- net EX_IO.IO3: now also J13.5 (Pin_5)
- net EX_IO.IO4: now also J13.6 (Pin_6)
- net EX_IO.IO5: now also J13.7 (Pin_7)
- net EX_IO.IO6: now also J13.8 (Pin_8)
- net EX_IO.IO7: now also J13.9 (Pin_9)
- net EX_IO.IO8: now also J13.10 (Pin_10)
- net EX_IO.IO9: now also J13.11 (Pin_11)
- net EX_IO.PWM0: now also J13.29 (Pin_29)
- net EX_IO.PWM1: now also J13.28 (Pin_28)
- net GND: now also H1.1, H2.1, H3.1, H4.1, J13.15 (Pin_15), J13.16 (Pin_16), J6.4 (Pin_4), J6.5 (Pin_5)
- net SWCLK: now also J6.2 (Pin_2)
- net SWDIO: now also J6.7 (Pin_7)
- net ~{RST}: now also J6.1 (Pin_1)
Other:
- note added: "安装孔"
- moved on the sheet: J5
