File: 通用型控制卡.kicad_sch (KiCad schematic)
At the start: 71 parts, among them J13 EXT, J2 HUB75_A, J3 HUB75_B, J4 PWR, J5 SWD_TC2030, J6 SWD_IDC, SW1 RESET, SW2 TST_KEY, U1 STM32H753IITx, U2 LD1117S33TR_SOT223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

Commit message: feat: 布局完成，正在布线
Parts:
- L1: footprint Inductor_SMD:L_12x12mm_H8mm -> wyh:L_12x12mm_H8mm
- Y1: footprint Crystal:Crystal_SMD_3225-4Pin_3.2x2.5mm_HandSoldering -> Crystal:Crystal_SMD_3225-4Pin_3.2x2.5mm
Changed lines of the file:
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@@
 		)
 	)
+	(global_label "~{RST}"
+		(shape output)
+		(at 44.45 54.61 180)
+		(fields_autoplaced yes)
+		(effects
+			(font
+				(size 1.27 1.27)
+			)
+			(justify right)
+		)
+		(property "Intersheetrefs" "${INTERSHEET_REFS}"
+			(at 38.0177 54.61 0)
+			(hide yes)
+			(show_name no)
+			(do_not_autoplace no)
+			(effects
+				(font
+					(size 1.27 1.27)
+				)
+				(justify right)
+			)
+		)
+	)
 	(global_label "RS485.TX2"
 		(shape output)
@@
 			)
 		)
-		(property "Footprint" "Crystal:Crystal_SMD_3225-4Pin_3.2x2.5mm_HandSoldering"
+		(property "Footprint" "Crystal:Crystal_SMD_3225-4Pin_3.2x2.5mm"
 			(at 185.42 111.76 0)
 			(hide yes)
@@
 		(unit 1)
 		(body_style 1)
-		(exclude_from_sim no)
+		(exclude_from_sim yes)
 		(in_bom no)
 		(on_board no)
@@
 		(unit 1)
 		(body_style 1)
-		(exclude_from_sim no)
+		(exclude_from_sim yes)
 		(in_bom no)
 		(on_board no)
@@
 			)
 		)
-		(property "Footprint" "Inductor_SMD:L_12x12mm_H8mm"
+		(property "Footprint" "wyh:L_12x12mm_H8mm"
 			(at 345.44 219.71 0)
 			(hide yes)
