File: 通用型控制卡.kicad_sch (KiCad schematic)
At the start: 71 parts, among them J13 EXT, J2 HUB75_A, J3 HUB75_B, J4 PWR, J5 SWD_TC2030, J6 SWD_IDC, SW1 RESET, SW2 TST_KEY, U1 STM32H753IITx, U2 LD1117S33TR_SOT223, U3 XL1509-ADJ, Y1 25Mhz, Y2 32768hz

Commit message: 根据BOM表调整部分元件封装
Parts:
- C24, C27: footprint Capacitor_SMD:CP_Elec_6.3x5.9 -> Capacitor_SMD:CP_Elec_4x5.7
- F1: footprint Fuse:Fuse_1206_3216Metric -> Fuse:Fuse_1812_4532Metric_Pad1.30x3.40mm_HandSolder
- J2: value HUB75_A -> HUB75_Socket
- J3: value HUB75_B -> HUB75_Socket
- SW1: value RESET -> KEY; 定义 (none) -> RESET
- SW2: value TST_KEY -> KEY; 定义 (none) -> TST_KEY
Changed lines of the file:
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@@
 			)
 		)
-		(property "Value" "HUB75_A"
+		(property "Value" "HUB75_Socket"
 			(at 352.298 156.21 0)
 			(show_name no)
@@
 			)
 		)
-		(property "Footprint" "Fuse:Fuse_1206_3216Metric"
+		(property "Footprint" "Fuse:Fuse_1812_4532Metric_Pad1.30x3.40mm_HandSolder"
 			(at 284.48 189.738 90)
 			(hide yes)
@@
 			)
 		)
-		(property "Value" "RESET"
+		(property "Value" "KEY"
 			(at 183.134 72.39 0)
+			(hide yes)
 			(show_name no)
 			(do_not_autoplace no)
@@
 			)
 		)
+		(property "定义" "RESET"
+			(at 183.134 72.39 0)
+			(show_name no)
+			(do_not_autoplace no)
+			(effects
+				(font
+					(size 1.27 1.27)
+				)
+			)
+		)
 		(pin "2"
 		)
@@
 			)
 		)
-		(property "Footprint" "Capacitor_SMD:CP_Elec_6.3x5.9"
+		(property "Footprint" "Capacitor_SMD:CP_Elec_4x5.7"
 			(at 328.6252 199.39 0)
 			(hide yes)
@@
 			)
 		)
-		(property "Value" "HUB75_B"
+		(property "Value" "HUB75_Socket"
 			(at 394.208 156.21 0)
 			(show_name no)
@@
 			)
 		)
-		(property "Value" "TST_KEY"
+		(property "Value" "KEY"
 			(at 271.78 151.638 0)
+			(hide yes)
 			(show_name no)
 			(do_not_autoplace no)
@@
 			)
 		)
+		(property "定义" "TST_KEY"
+			(at 271.78 151.384 0)
+			(show_name no)
+			(do_not_autoplace no)
+			(effects
+				(font
+					(size 1.27 1.27)
+				)
+			)
+		)
 		(pin "1"
 		)
@@
 			)
 		)
-		(property "Footprint" "Capacitor_SMD:CP_Elec_6.3x5.9"
+		(property "Footprint" "Capacitor_SMD:CP_Elec_4x5.7"
 			(at 375.6152 199.39 0)
 			(hide yes)

Commit message: fix: 修改了485芯片的封装，添加了保险丝的封装
Parts:
- F1: footprint Fuse:Fuse_1812_4532Metric_Pad1.30x3.40mm_HandSolder -> wyh:Fuse_1812_4532Metric_Pad1.30x3.40mm_HandSolder
Changed lines of the file:
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@@
 			)
 		)
-		(property "Footprint" "Fuse:Fuse_1812_4532Metric_Pad1.30x3.40mm_HandSolder"
+		(property "Footprint" "wyh:Fuse_1812_4532Metric_Pad1.30x3.40mm_HandSolder"
 			(at 284.48 189.738 90)
 			(hide yes)
