File: storage.kicad_sch (KiCad schematic)
At the start: 15 parts, among them J13 Micro_SD_Card, U10 IP4220CZ6, U8 24LC08, U9 IP4220CZ6

Commit message: style: 修改图框
Other:
- title: (none) -> 存储组件
Changed lines of the file:
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@@
 	(paper "A5")
 	(title_block
-		(date "2026-06-08")
+		(title "存储组件")
+		(date "2026-06-10")
+		(rev "V0.0.1")
 		(company "重庆创迪科技发展有限公司")
 	)

Commit message: feat: 添加了安装孔
Parts:
- renumbered J13 to J12
Changed lines of the file:
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@@
 		(in_pos_files yes)
 		(dnp no)
-		(property "Reference" "#PWR068"
+		(property "Reference" "#PWR067"
 			(at 50.8 39.37 0)
 			(hide yes)
@@
 			(project "通用型控制卡"
 				(path "/265862a2-6b57-40ac-b33f-86ad5d011aff"
-					(reference "#PWR068")
+					(reference "#PWR067")
 					(unit 1)
 				)
@@
 		(in_pos_files yes)
 		(dnp no)
-		(property "Reference" "#PWR073"
+		(property "Reference" "#PWR072"
 			(at 128.27 88.9 0)
 			(hide yes)
@@
 			(project "通用型控制卡"
 				(path "/265862a2-6b57-40ac-b33f-86ad5d011aff"
-					(reference "#PWR073")
+					(reference "#PWR072")
 					(unit 1)
 				)
@@
 		(in_pos_files yes)
 		(dnp no)
-		(property "Reference" "#PWR071"
+		(property "Reference" "#PWR070"
 			(at 128.27 63.5 0)
 			(hide yes)
@@
 			(project "通用型控制卡"
 				(path "/265862a2-6b57-40ac-b33f-86ad5d011aff"
-					(reference "#PWR071")
+					(reference "#PWR070")
 					(unit 1)
 				)
@@
 		(dnp no)
 		(fields_autoplaced yes)
-		(property "Reference" "J13"
+		(property "Reference" "J12"
 			(at 167.005 25.4 0)
 			(show_name no)
@@
 			(project "通用型控制卡"
 				(path "/265862a2-6b57-40ac-b33f-86ad5d011aff"
-					(reference "J13")
+					(reference "J12")
 					(unit 1)
 				)
@@
 		(in_pos_files yes)
 		(dnp no)
-		(property "Reference" "#PWR067"
+		(property "Reference" "#PWR066"
 			(at 149.86 30.48 0)
 			(hide yes)
@@
 			(project "通用型控制卡"
 				(path "/265862a2-6b57-40ac-b33f-86ad5d011aff"
-					(reference "#PWR067")
+					(reference "#PWR066")
 					(unit 1)
 				)
@@
 		(in_pos_files yes)
 		(dnp no)
-		(property "Reference" "#PWR066"
+		(property "Reference" "#PWR065"
 			(at 130.81 25.4 0)
 			(hide yes)
@@
 			(project "通用型控制卡"
 				(path "/265862a2-6b57-40ac-b33f-86ad5d011aff"
-					(reference "#PWR066")
+					(reference "#PWR065")
 					(unit 1)
 				)
@@
 		(in_pos_files yes)
 		(dnp no)
-		(property "Reference" "#PWR069"
+		(property "Reference" "#PWR068"
 			(at 142.24 63.5 0)
 			(hide yes)
@@
 			(project "通用型控制卡"
 				(path "/265862a2-6b57-40ac-b33f-86ad5d011aff"
-					(reference "#PWR069")
+					(reference "#PWR068")
 					(unit 1)
 				)
@@
 		(in_pos_files yes)
 		(dnp no)
-		(property "Reference" "#PWR070"
+		(property "Reference" "#PWR069"
 			(at 62.23 66.04 0)
 			(hide yes)
@@
 			(project "通用型控制卡"
 				(path "/265862a2-6b57-40ac-b33f-86ad5d011aff"
-					(reference "#PWR070")
+					(reference "#PWR069")
 					(unit 1)
 				)
@@
 		(in_pos_files yes)
 		(dnp no)
-		(property "Reference" "#PWR072"
+		(property "Reference" "#PWR071"
 			(at 187.96 67.31 0)
 			(hide yes)
@@
 			(project "通用型控制卡"
 				(path "/265862a2-6b57-40ac-b33f-86ad5d011aff"
-					(reference "#PWR072")
-					(unit 1)
-				)
+					(reference "#PWR071")
+					(unit 1)
+				)

Commit message: feat: 布局完成，正在布线
Parts:
- J12: footprint Connector_Card:microSD_HC_Molex_47219-2001 -> wyh:microSD_HC_Molex_47219-2001
Connections:
- net EEPROM.SCL: now also R36.2
- net EEPROM.SDA: no longer R36.2
Other:
- note added: "Tips: 4根Data信号线徐要走等长，长度控制在50mil以内"
- moved on the sheet: C58
Changed lines of the file:
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@@
+		)
+	)
+	(text "Tips: 4根Data信号线徐要走等长，长度控制在50mil以内"
+		(exclude_from_sim no)
+		(at 160.274 66.802 0)
+		(effects
+			(font
+				(size 1.27 1.27)
+			)
 		)
 	)
@@
 	)
 	(junction
-		(at 38.1 36.83)
+		(at 38.1 49.53)
 		(diameter 0)
 		(color 0 0 0 0)
 	)
 	(junction
-		(at 50.8 40.64)
+		(at 38.1 36.83)
 		(diameter 0)
 		(color 0 0 0 0)
@@
 	)
 	(junction
-		(at 38.1 46.99)
-		(diameter 0)
-		(color 0 0 0 0)
-	)
-	(junction
 		(at 115.57 41.91)
 		(diameter 0)
@@
 	(wire
 		(pts
+			(xy 38.1 49.53) (xy 40.64 49.53)
+		)
+		(stroke
+			(width 0)
+			(type default)
+		)
+	)
+	(wire
+		(pts
 			(xy 92.71 41.91) (xy 115.57 41.91)
 		)
@@
 	(wire
 		(pts
-			(xy 53.34 40.64) (xy 50.8 40.64)
+			(xy 53.34 36.83) (xy 50.8 36.83)
 		)
 		(stroke
@@
 	(wire
 		(pts
-			(xy 50.8 36.83) (xy 50.8 40.64)
+			(xy 50.8 36.83) (xy 50.8 41.91)
 		)
 		(stroke
@@
 		)
 	)
-	(wire
-		(pts
-			(xy 38.1 45.72) (xy 38.1 46.99)
-		)
-		(stroke
-			(width 0)
-			(type default)
-		)
-	)
 	(polyline
 		(pts
@@
 	(wire
 		(pts
-			(xy 60.96 40.64) (xy 62.23 40.64)
-		)
-		(stroke
-			(width 0)
-			(type default)
-		)
-	)
-	(wire
-		(pts
-			(xy 31.75 46.99) (xy 38.1 46.99)
-		)
-		(stroke
-			(width 0)
-			(type default)
-		)
-	)
-	(wire
-		(pts
-			(xy 38.1 46.99) (xy 40.64 46.99)
-		)
-		(stroke
-			(width 0)
-			(type default)
-		)
-	)
-	(wire
-		(pts
-			(xy 30.48 49.53) (xy 40.64 49.53)
+			(xy 60.96 36.83) (xy 62.23 36.83)
+		)
+		(stroke
+			(width 0)
+			(type default)
+		)
+	)
+	(wire
+		(pts
+			(xy 31.75 46.99) (xy 40.64 46.99)
+		)
+		(stroke
+			(width 0)
+			(type default)
+		)
+	)
+	(wire
+		(pts
+			(xy 30.48 49.53) (xy 38.1 49.53)
 		)
 		(stroke
@@
 	(wire
 		(pts
+			(xy 38.1 45.72) (xy 38.1 49.53)
+		)
+		(stroke
+			(width 0)
+			(type default)
+		)
+	)
+	(wire
+		(pts
 			(xy 115.57 22.86) (xy 115.57 24.13)
 		)
@@
 	(wire
 		(pts
-			(xy 62.23 40.64) (xy 62.23 46.99)
+			(xy 62.23 36.83) (xy 62.23 46.99)
 		)
 		(stroke
@@
 		(pts
 			(xy 102.87 22.86) (xy 109.22 22.86)
-		)
-		(stroke
-			(width 0)
-			(type default)
-		)
-	)
-	(wire
-		(pts
-			(xy 50.8 40.64) (xy 50.8 41.91)
 		)
 		(stroke
@@
 		(dnp no)
 		(property "Reference" "R35"
-			(at 26.67 41.148 0)
+			(at 26.67 40.894 0)
 			(show_name no)
 			(do_not_autoplace no)
@@
 			)
 		)
-		(property "Footprint" "Connector_Card:microSD_HC_Molex_47219-2001"
+		(property "Footprint" "wyh:microSD_HC_Molex_47219-2001"
 			(at 195.58 36.83 0)
 			(hide yes)
@@
 	(symbol
 		(lib_id "Device:C")
-		(at 57.15 40.64 270)
+		(at 57.15 36.83 270)
 		(mirror x)
 		(unit 1)
@@
 		(dnp no)
 		(property "Reference" "C58"
-			(at 55.372 35.306 90)
+			(at 55.372 31.496 90)
 			(show_name no)
 			(do_not_autoplace no)
@@
 		)
 		(property "Value" "100nF"
-			(at 54.102 37.338 90)
+			(at 54.102 33.528 90)
 			(show_name no)
 			(do_not_autoplace no)
@@
 		)
 		(property "Footprint" "Capacitor_SMD:C_0402_1005Metric_Pad0.74x0.62mm_HandSolder"
-			(at 53.34 39.6748 0)
+			(at 53.34 35.8648 0)
 			(hide yes)
 			(show_name no)
@@
 		)
 		(property "Datasheet" ""
-			(at 57.15 40.64 0)
+			(at 57.15 36.83 0)
 			(hide yes)
 			(show_name no)
@@
 		)
 		(property "Description" "Unpolarized capacitor"
-			(at 57.15 40.64 0)
-			(hide yes)
-			(show_name no)
+			(at 57.15 36.83 0)
+			(hide yes)
+			(show_name no)
