File: storage.kicad_sch (KiCad schematic)
At the start: 15 parts, among them J12 Micro_SD_Card, U10 IP4220CZ6, U8 24LC08, U9 IP4220CZ6

Commit message: 根据BOM表调整部分元件封装
Parts:
- C57: footprint Capacitor_SMD:C_0402_1005Metric_Pad0.74x0.62mm_HandSolder -> Capacitor_SMD:C_0603_1608Metric_Pad1.08x0.95mm_HandSolder
Changed lines of the file:
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@@
 			)
 		)
-		(property "Footprint" "Capacitor_SMD:C_0402_1005Metric_Pad0.74x0.62mm_HandSolder"
+		(property "Footprint" "Capacitor_SMD:C_0603_1608Metric_Pad1.08x0.95mm_HandSolder"
 			(at 143.51 29.5148 0)
 			(hide yes)
