File: 通用型控制卡.kicad_pcb (KiCad board)
At the start: 4 copper layers, 100 x 100 mm, 135 parts, among them J1 EXT, J10 RS232_1, J11 RS232_2, J12 RJ45_Hanrun_HR911105A_Horizon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, J13 Micro_SD_Card, J2 HUB75_A, J3 HUB75_B, J4 PWR, J5 SWD_TC2030, J6 SWD_IDC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

Commit message: feat: 添加了安装孔
Parts:
- removed J1: EXT, Connector_JST:JST_PUD_B32B-PUDSS_2x16_P2.00mm_Vertical
- removed the J7 at (91.3, -118.2)
- added H1: MountingHole_Pad, MountingHole:MountingHole_3.2mm_M3_Pad, F.Cu at (4.97, -95.0)
- added H2: MountingHole_Pad, MountingHole:MountingHole_3.2mm_M3_Pad, F.Cu at (95.0, -95.0)
- added H3: MountingHole_Pad, MountingHole:MountingHole_3.2mm_M3_Pad, F.Cu at (95.0, -5.00)
- added H4: MountingHole_Pad, MountingHole:MountingHole_3.2mm_M3_Pad, F.Cu at (5.00, -5.00)
- added J12: Micro_SD_Card, Connector_Card:microSD_HC_Molex_47219-2001, B.Cu at (9.00, -77.4)
- C25, C26, C29, C30, C31, C32, C56, C57, D4, D5, D6, F1, R10, R29, R30, R31, R32, R33, R34, R8, R9, U10, U3, U9: moved to B.Cu
- J13: value Micro_SD_Card -> EXT; footprint Connector_Card:microSD_HC_Molex_47219-2001 -> Connector_IDC:IDC-Header_2x15_P2.54mm_Vertical
- J6: footprint Connector_IDC:IDC-Header_2x03_P2.54mm_Vertical -> Connector_IDC:IDC-Header_2x04_P2.54mm_Vertical
- moved D5 104.8 mm to (18.9, -62.3), turned to 180 degrees
- moved U2 99.5 mm to (7.80, -66.0)
- moved J4 95.5 mm to (5.50, -54.4), turned to -90 degrees
- moved R30 88.1 mm to (3.96, -67.4), turned to -90 degrees
- moved R32 88.1 mm to (7.94, -67.4), turned to -90 degrees
- moved R29 88.1 mm to (1.97, -67.4), turned to -90 degrees
- moved R31 88.1 mm to (5.95, -67.4), turned to -90 degrees
- moved R33 88.1 mm to (9.93, -67.4), turned to -90 degrees
- moved R34 88.1 mm to (11.9, -67.4), turned to -90 degrees
- moved L1 86.3 mm to (15.9, -52.8)
- moved C24 78.7 mm to (22.7, -65.0)
- moved C27 74.9 mm to (27.0, -53.0), turned to 90 degrees
- moved C25 74.6 mm to (11.7, -63.3), turned to 180 degrees
- moved C26 74.6 mm to (11.7, -60.8), turned to 180 degrees
- moved C30 74.6 mm to (11.7, -55.8), turned to 180 degrees
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- renumbered J11 to J10, J12 to J11, J8 to J7, J9 to J8, J10 to J9
Connections:
- J13 pad 1: SDMMC.D2 -> +5V
- J13 pad 2: SDMMC.D3 -> /通用型控制卡/EX_IO.IO0
- J13 pad 3: SDMMC.CMD -> /通用型控制卡/EX_IO.IO1
- J13 pad 4: +3V3 -> /通用型控制卡/EX_IO.IO2
- J13 pad 5: SDMMC.CK -> /通用型控制卡/EX_IO.IO3
- J13 pad 6: GND -> /通用型控制卡/EX_IO.IO4
- J13 pad 7: SDMMC.D0 -> /通用型控制卡/EX_IO.IO5
- J13 pad 8: SDMMC.D1 -> /通用型控制卡/EX_IO.IO6
- J6 pad 3: GND -> /通用型控制卡/DBG_MCU_RX
- J6 pad 5: /通用型控制卡/SWDIO -> GND
- J6 pad 6: +3V3 -> /通用型控制卡/DBG_MCU_TX
Other:
- rule pad_to_mask_clearance: 0 -> 0.07

Commit message: feat: 布局完成，正在布线
Parts:
- C25, C26, C45, C46, C47, C51, C52, C53, C54, C55, D5, D6, FB1, R10, R25, R26, R27, R8, R9: moved to F.Cu
- C41, D10, D11, D12, D7, D8, D9, R15, R16, R17, R18, R23, R3, U4, U5, U6: moved to B.Cu
- J11: footprint Connector_RJ:RJ45_Hanrun_HR911105A_Horizontal -> wyh:RJ45_Hanrun_HR911105A_Horizontal
- J12: footprint Connector_Card:microSD_HC_Molex_47219-2001 -> wyh:microSD_HC_Molex_47219-2001; moved to F.Cu
- L1: footprint Inductor_SMD:L_12x12mm_H8mm -> wyh:L_12x12mm_H8mm
- U7: footprint Package_DFN_QFN:VQFN-24-1EP_4x4mm_P0.5mm_EP2.5x2.5mm_ThermalVias -> wyh:VQFN-24-1EP_4x4mm_P0.5mm_EP2.5x2.5mm_ThermalVias
- Y1, Y3: footprint Crystal:Crystal_SMD_3225-4Pin_3.2x2.5mm_HandSoldering -> Crystal:Crystal_SMD_3225-4Pin_3.2x2.5mm
- moved R9 64.3 mm to (62.5, -85.1), turned to 90 degrees
- moved SW1 60.7 mm to (90.6, -75.0)
- moved D6 53.3 mm to (60.7, -85.1), turned to -90 degrees
- moved C17 51.0 mm to (86.2, -73.9), turned to -90 degrees
- moved C40 35.5 mm to (76.9, -26.7), turned to 90 degrees
- moved D8 34.2 mm to (84.9, -60.0), turned to 180 degrees
- moved C51 31.2 mm to (15.3, -30.9), turned to -90 degrees
- moved R3 30.9 mm to (49.1, -38.1), turned to -135 degrees
- moved C52 30.5 mm to (13.5, -30.9), turned to -90 degrees
- moved C42 30.3 mm to (81.6, -32.0), turned to 0 degrees
- moved C53 29.9 mm to (11.7, -30.9), turned to -90 degrees
- moved C43 29.9 mm to (78.4, -32.5), turned to 90 degrees
- moved C44 29.5 mm to (83.5, -32.7), turned to 90 degrees
- moved C54 29.2 mm to (9.90, -30.9), turned to -90 degrees
- moved C55 28.5 mm to (8.10, -30.9), turned to -90 degrees
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Connections:
- C17 pad 2: /通用型控制卡/~{RST} -> ~{RST}
- J5 pad 3: /通用型控制卡/~{RST} -> ~{RST}
- J6 pad 1: /通用型控制卡/~{RST} -> ~{RST}
- R20 pad 2: /ethernet/RJ45_TX- -> /ethernet/RJ45_RX+
- R3 pad 2: /通用型控制卡/~{RST} -> ~{RST}
- R36 pad 2: EEPROM.SDA -> EEPROM.SCL
- SW1 pad 2: /通用型控制卡/~{RST} -> ~{RST}
- U1 pad 31: /通用型控制卡/~{RST} -> ~{RST}
- U7 pad 15: /ethernet/~{RST} -> ~{RST}
Routing:
- net ~{RST}: track 0.00 -> 132.0 mm, vias 0 -> 5
- net /通用型控制卡/HUB75.D: track 0.00 -> 103.9 mm, vias 0 -> 3
- net /通用型控制卡/HUB75.C: track 0.00 -> 103.5 mm, vias 0 -> 3
- net /通用型控制卡/HUB75.B: track 0.00 -> 101.6 mm, vias 0 -> 3
- net /通用型控制卡/HUB75.A: track 0.00 -> 100.9 mm, vias 0 -> 3
- net /通用型控制卡/HUB75.LAT: track 0.00 -> 98.6 mm, vias 0 -> 3
- net /通用型控制卡/HUB75.CLK: track 0.00 -> 98.1 mm, vias 0 -> 3
- net /通用型控制卡/HUB75.~{OE}: track 0.00 -> 95.9 mm, vias 0 -> 3
- net SDMMC.D1: track 0.00 -> 88.1 mm, vias 0 -> 1
- net SDMMC.CK: track 0.00 -> 87.8 mm, vias 0 -> 1
- net SDMMC.CMD: track 0.00 -> 87.5 mm, vias 0 -> 1
- net SDMMC.D3: track 0.00 -> 87.2 mm, vias 0 -> 3
- net SDMMC.D0: track 0.00 -> 85.0 mm, vias 0 -> 3
- net /通用型控制卡/EX_IO.PWM0: track 0.00 -> 84.7 mm, vias 0 -> 3
- net SDMMC.D2: track 0.00 -> 81.4 mm, vias 0 -> 5
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- added copper zone on F.Cu, net +3V3
- added copper zone on B.Cu, net +5V
- added copper zone on F.Cu, net +5V
- added copper zone on B.Cu, net 4V5~16V
- added copper zone on F.Cu, net 4V5~16V
- added copper zone on B.Cu, net GND
- added copper zone on F.Cu, net GND
- added copper zone on In1.Cu, net GND
- added copper zone on In2.Cu, net GND
- added copper zone on B.Cu, net Net-(J4-Pin_1)
Other:
- rule pad_to_mask_clearance: 0.07 -> 0.2
